File: Micro_Air_Vehicle.kicad_sch (KiCad schematic)
At the start: 52 parts, among them IC2 CONMHF1-SMD-G-T, SW2 SW_Push, SW3 SW_Push, U1 ESP32-S3, U2 FLASH, U3 PSRAM, Y1 40MHz Quarz

Commit message: 
Parts:
- D3, D4, D5, D6: footprint LED_THT:LED_D3.0mm -> LED_SMD:LED_1206_3216Metric
Changed lines of the file:
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@@
 			)
 		)
-		(property "Footprint" "LED_THT:LED_D3.0mm"
+		(property "Footprint" "LED_SMD:LED_1206_3216Metric"
 			(at 237.49 62.23 0)
 			(hide yes)
@@
 			)
 		)
-		(property "Footprint" "LED_THT:LED_D3.0mm"
+		(property "Footprint" "LED_SMD:LED_1206_3216Metric"
 			(at 237.49 88.9 0)
 			(hide yes)
@@
 			)
 		)
-		(property "Footprint" "LED_THT:LED_D3.0mm"
+		(property "Footprint" "LED_SMD:LED_1206_3216Metric"
 			(at 237.49 71.12 0)
 			(hide yes)
@@
 			)
 		)
-		(property "Footprint" "LED_THT:LED_D3.0mm"
+		(property "Footprint" "LED_SMD:LED_1206_3216Metric"
 			(at 237.49 80.01 0)
 			(hide yes)
