File: Micro_Air_Vehicle.kicad_pcb (KiCad board)
At the start: 4 copper layers, 91.1 x 91.1 mm, 173 parts, among them IC1 BMI270, IC2 CONMHF1-SMD-G-T, J2 Akku Stecker, J3 Motor1, J4 Motor2, J5 Motor3, J6 Motor4, J7 USB4800-03-A, SW1 SW_SPDT, SW2 SW_Push, SW3 SW_Push, U1 ESP32-S3, U10 DRV8311P, U11 LMV339, U12 LMV339, U13 LMV339, U14 LMV339, U2 FLASH, U3 PSRAM, U4 TPD2EUSB30A, U5 BQ24074RGT, U6 TPS63031DSK, U7 DRV8311P, U8 DRV8311P, U9 DRV8311P, Y1 40MHz Quarz

Commit message: 
Parts:
- added R62: 10k, Resistor_SMD:R_0603_1608Metric, B.Cu at (239.8, 73.5)
- C22, C23: value DNP -> C
- D3, D4, D5, D6: footprint LED_THT:LED_D3.0mm -> LED_SMD:LED_1206_3216Metric
Routing:
- net Net-(U1-GPIO0): track 13.7 -> 15.9 mm

Commit message: Test
Parts:
- moved D5 9.22 mm to (271.6, 21.6)
Routing:
- net Net-(D5-A): track 0.00 -> 37.3 mm
Changed lines of the file:
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@@
 	(footprint "LED_SMD:LED_1206_3216Metric"
 		(layer "F.Cu")
-		(at 264.96 28)
+		(at 271.6 21.6)
 		(descr "LED SMD 1206 (3216 Metric), square (rectangular) end terminal, IPC-7351 nominal, (Body size source: http://www.tortai-tech.com/upload/download/2011102023233369053.pdf)")
 		(tags "LED")
@@
 	)
 	(segment
+		(start 270.612605 33.599397)
+		(end 271.153144 33.034778)
+		(width 0.2)
+		(layer "F.Cu")
+		(net "Net-(D5-A)")
+	)
+	(segment
+		(start 270.599232 33.599688)
+		(end 270.612605 33.599397)
+		(width 0.2)
+		(layer "F.Cu")
+		(net "Net-(D5-A)")
+	)
+	(segment
+		(start 270 38.6)
+		(end 270 34.19892)
+		(width 0.2)
+		(layer "F.Cu")
+		(net "Net-(D5-A)")
+	)
+	(segment
+		(start 270 34.19892)
+		(end 270.599232 33.599688)
+		(width 0.2)
+		(layer "F.Cu")
+		(net "Net-(D5-A)")
+	)
+	(segment
+		(start 272.6 34.481634)
+		(end 272.6 45.4)
+		(width 0.2)
+		(layer "F.Cu")
+		(net "Net-(D5-A)")
+	)
+	(segment
+		(start 273 35.6)
+		(end 270 38.6)
+		(width 0.2)
+		(layer "F.Cu")
+		(net "Net-(D5-A)")
+	)
+	(segment
+		(start 273 21.6)
+		(end 273 35.6)
+		(width 0.2)
+		(layer "F.Cu")
+		(net "Net-(D5-A)")
+	)
+	(segment
+		(start 271.153144 33.034778)
+		(end 272.6 34.481634)
+		(width 0.2)
+		(layer "F.Cu")
+		(net "Net-(D5-A)")
+	)
+	(segment
 		(start 232.962352 69.75)
 		(end 233.262352 69.45)
@@
 	)
 	(segment
-		(start 238.55 66.2)
-		(end 238.55 66.85)
-		(width 0.2)
-		(layer "B.Cu")
-		(net "Net-(U1-GPIO0)")
-	)
-	(segment
-		(start 231.55 66.95)
-		(end 232.75 65.75)
-		(width 0.2)
-		(layer "B.Cu")
-		(net "Net-(U1-GPIO0)")
-	)
-	(segment
-		(start 238.55 70.95)
-		(end 239.77 72.17)
-		(width 0.2)
-		(layer "B.Cu")
-		(net "Net-(U1-GPIO0)")
-	)
-	(segment
-		(start 230.3 66.95)
-		(end 231.55 66.95)
-		(width 0.2)
-		(layer "B.Cu")
-		(net "Net-(U1-GPIO0)")
-	)
-	(segment
-		(start 232.75 65.75)
-		(end 238.1 65.75)
-		(width 0.2)
-		(layer "B.Cu")
-		(net "Net-(U1-GPIO0)")
-	)
-	(segment
-		(start 238.55 70.95)
-		(end 238.55 66.85)
-		(width 0.2)
-		(layer "B.Cu")
-		(net "Net-(U1-GPIO0)")
-	)
-	(segment
-		(start 238.1 65.75)
-		(end 238.55 66.2)
-		(width 0.2)
-		(layer "B.Cu")
-		(net "Net-(U1-GPIO0)")
-	)
-	(segment
-		(start 239.77 72.17)
-		(end 239.77 72.655)
-		(width 0.2)
-		(layer "B.Cu")
-		(net "Net-(U1-GPIO0)")
-	)
-	(segment
 		(start 218.95 71.46)
 		(end 218.96 71.45)
@@
 	)
 	(segment
+		(start 238.55 66.2)
+		(end 238.55 66.85)
+		(width 0.2)
+		(layer "B.Cu")
+		(net "Net-(U1-GPIO0)")
+	)
+	(segment
+		(start 231.55 66.95)
+		(end 232.75 65.75)
+		(width 0.2)
+		(layer "B.Cu")
+		(net "Net-(U1-GPIO0)")
+	)
+	(segment
+		(start 238.55 70.95)
+		(end 239.77 72.17)
+		(width 0.2)
+		(layer "B.Cu")
+		(net "Net-(U1-GPIO0)")
+	)
+	(segment
+		(start 230.3 66.95)
+		(end 231.55 66.95)
+		(width 0.2)
+		(layer "B.Cu")
+		(net "Net-(U1-GPIO0)")
+	)
+	(segment
+		(start 232.75 65.75)
+		(end 238.1 65.75)
+		(width 0.2)
+		(layer "B.Cu")
+		(net "Net-(U1-GPIO0)")
+	)
+	(segment
+		(start 238.55 70.95)
+		(end 238.55 66.85)
+		(width 0.2)
+		(layer "B.Cu")
+		(net "Net-(U1-GPIO0)")
+	)
+	(segment
+		(start 238.1 65.75)
+		(end 238.55 66.2)
+		(width 0.2)
+		(layer "B.Cu")
+		(net "Net-(U1-GPIO0)")
+	)
+	(segment
+		(start 239.77 72.17)
+		(end 239.77 72.655)
+		(width 0.2)
+		(layer "B.Cu")
+		(net "Net-(U1-GPIO0)")
+	)
+	(segment

Commit message: Test
Routing:
- net Net-(D5-A): track 37.3 -> 0.00 mm
Changed lines of the file:
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@@
-	)
-	(segment
-		(start 270.612605 33.599397)
-		(end 271.153144 33.034778)
-		(width 0.2)
-		(layer "F.Cu")
-		(net "Net-(D5-A)")
-	)
-	(segment
-		(start 270.599232 33.599688)
-		(end 270.612605 33.599397)
-		(width 0.2)
-		(layer "F.Cu")
-		(net "Net-(D5-A)")
-	)
-	(segment
-		(start 270 38.6)
-		(end 270 34.19892)
-		(width 0.2)
-		(layer "F.Cu")
-		(net "Net-(D5-A)")
-	)
-	(segment
-		(start 270 34.19892)
-		(end 270.599232 33.599688)
-		(width 0.2)
-		(layer "F.Cu")
-		(net "Net-(D5-A)")
-	)
-	(segment
-		(start 272.6 34.481634)
-		(end 272.6 45.4)
-		(width 0.2)
-		(layer "F.Cu")
-		(net "Net-(D5-A)")
-	)
-	(segment
-		(start 273 35.6)
-		(end 270 38.6)
-		(width 0.2)
-		(layer "F.Cu")
-		(net "Net-(D5-A)")
-	)
-	(segment
-		(start 273 21.6)
-		(end 273 35.6)
-		(width 0.2)
-		(layer "F.Cu")
-		(net "Net-(D5-A)")
-	)
-	(segment
-		(start 271.153144 33.034778)
-		(end 272.6 34.481634)
-		(width 0.2)
-		(layer "F.Cu")
-		(net "Net-(D5-A)")
 	)
 	(segment

Commit message: IMU
Parts:
- moved C29 91.3 mm to (205.1, 47.1)
- moved C62 91.3 mm to (201.6, 40.8)
- moved C63 91.3 mm to (199.4, 38.7)
- moved C64 91.3 mm to (198.4, 44.0)
- moved R25 91.3 mm to (197.3, 36.6)
- moved R28 91.3 mm to (197.3, 43.0)
- moved U7 91.3 mm to (203.8, 46.9)
- moved C28 91.3 mm to (206.4, 48.2)
- moved C30 91.3 mm to (207.5, 49.4)
- moved C31 91.3 mm to (203.6, 45.7)
- moved C33 91.3 mm to (205.5, 44.4)
- moved C34 91.3 mm to (206.7, 44.9)
- moved J3 91.3 mm to (195.8, 33.8)
- moved R19 91.3 mm to (200.5, 39.7)
- moved R26 91.3 mm to (198.3, 37.7)
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Routing:
- net IMU_CS: track 1.12 -> 24.0 mm
- net IMU_MOSI: track 2.26 -> 16.5 mm, vias 1 -> 2
- net IMU_INT: track 0.00 -> 11.9 mm, vias 0 -> 1
- net IMU_SCK: track 8.76 -> 20.0 mm
- net IMU_MISO: track 10.2 -> 16.5 mm

Commit message: 
Routing:
- net GND: track 109.1 -> 108.2 mm
- net BAT+: track 16.3 -> 15.6 mm
- net SYS_OUT: track 14.0 -> 14.7 mm
Changed lines of the file:
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@@
 		(tags "capacitor")
 		(property "Reference" "C47"
-			(at -104.054902 46.441593 135)
+			(at 0.280026 -1.315219 135)
 			(layer "F.SilkS")
 			(effects
@@
 		(tags "inductor")
 		(property "Reference" "L5"
-			(at -56.3 2.3 90)
+			(at 1.815 0.32 90)
 			(layer "B.SilkS")
 			(effects
@@
 		(tags "tactile switch kmr2")
 		(property "Reference" "SW2"
-			(at -0.33 65.875 90)
+			(at 0 2.44 90)
 			(layer "B.SilkS")
 			(effects
@@
 	)
 	(segment
-		(start 235.4 71.85)
-		(end 237.15 71.85)
+		(start 186.775 67.851886)
+		(end 186.775 68.235)
 		(width 0.2)
 		(layer "F.Cu")
@@
 	)
 	(segment
-		(start 205.671751 46.403249)
-		(end 205.721751 46.403249)
+		(start 237.65 72.35)
+		(end 237.15 72.35)
 		(width 0.2)
 		(layer "F.Cu")
@@
 	)
 	(segment
-		(start 224 53.75)
-		(end 224 54.2)
+		(start 186.775 67.85)
+		(end 186.775 67.455)
+		(width 0.2)
+		(layer "F.Cu")
+		(net "GND")
+	)
+	(segment
+		(start 205.671751 46.403249)
+		(end 205.721751 46.403249)
 		(width 0.2)
 		(layer "F.Cu")
@@
 	)
 	(segment
+		(start 186.775 67.455)
+		(end 186.6825 67.3625)
+		(width 0.2)
+		(layer "F.Cu")
+		(net "GND")
+	)
+	(segment
 		(start 179.825 68.9)
 		(end 179.825 67.5)
@@
 	)
 	(segment
-		(start 186.264386 68.3625)
-		(end 185.8375 68.3625)
-		(width 0.2)
-		(layer "F.Cu")
-		(net "GND")
-	)
-	(segment
 		(start 183.625 63.65)
 		(end 185.225 63.65)
@@
 	)
 	(segment
-		(start 224 54.2)
-		(end 223.9 54.3)
+		(start 195.3 43.928805)
+		(end 195.3 45.525)
 		(width 0.2)
 		(layer "F.Cu")
@@
 	)
 	(segment
-		(start 195.3 43.928805)
-		(end 195.3 45.525)
+		(start 224 54.2)
+		(end 223.9 54.3)
 		(width 0.2)
 		(layer "F.Cu")
@@
 	)
 	(segment
-		(start 223.6 53.15)
-		(end 223.6 53.35)
-		(width 0.2)
-		(layer "F.Cu")
-		(net "GND")
-	)
-	(segment
 		(start 196.461522 45.525)
 		(end 197.680761 44.305761)
@@
 	)
 	(segment
-		(start 186.2875 67.3625)
-		(end 185.8375 67.3625)
-		(width 0.2)
-		(layer "F.Cu")
-		(net "GND")
-	)
-	(segment
 		(start 233.075 71.525)
 		(end 233.4 71.85)
@@
 	)
 	(segment
-		(start 237.15 71.85)
-		(end 237.65 72.35)
+		(start 223.6 53.15)
+		(end 224 53.55)
 		(width 0.2)
 		(layer "F.Cu")
@@
 	)
 	(segment
-		(start 223.6 53.35)
-		(end 224 53.75)
+		(start 186.775 68.235)
+		(end 186.6475 68.3625)
 		(width 0.2)
 		(layer "F.Cu")
@@
 	)
 	(segment
+		(start 186.6475 68.3625)
+		(end 185.8375 68.3625)
+		(width 0.2)
+		(layer "F.Cu")
+		(net "GND")
+	)
+	(segment
 		(start 196.301902 42.926903)
 		(end 195.3 43.928805)
@@
 	)
 	(segment
-		(start 228.038 71.513)
-		(end 227.838 71.713)
+		(start 237.15 72.35)
+		(end 236.7 72.8)
 		(width 0.2)
 		(layer "F.Cu")
@@
 	)
 	(segment
-		(start 226.838 69.513)
-		(end 227.338 69.513)
+		(start 228.038 71.513)
+		(end 227.838 71.713)
 		(width 0.2)
 		(layer "F.Cu")
@@
 	)
 	(segment
-		(start 186.775 67.85)
-		(end 186.2875 67.3625)
+		(start 226.838 69.513)
+		(end 227.338 69.513)
 		(width 0.2)
 		(layer "F.Cu")
@@
 	)
 	(segment
-		(start 186.775 67.851886)
-		(end 186.264386 68.3625)
+		(start 230 53.15)
+		(end 230 53.45)
 		(width 0.2)
 		(layer "F.Cu")
@@
 	)
 	(segment
-		(start 230 53.15)
-		(end 230 53.45)
+		(start 230.15 55.8)
+		(end 230.15 54.35)
 		(width 0.2)
 		(layer "F.Cu")
@@
 	)
 	(segment
-		(start 230.15 55.8)
-		(end 230.15 54.35)
+		(start 186.6825 67.3625)
+		(end 185.8375 67.3625)
 		(width 0.2)
 		(layer "F.Cu")
@@
 	)
 	(segment
+		(start 224 53.55)
+		(end 224 54.2)
+		(width 0.2)
+		(layer "F.Cu")
+		(net "GND")
+	)
+	(segment
 		(start 185.225 63.65)
 		(end 187.575 66)
@@
 	)
 	(segment
-		(start 184.625 69.575)
-		(end 184.625 70.75)
-		(width 0.2)
-		(layer "F.Cu")
-		(net "BAT+")
-	)
-	(segment
 		(start 191.975 68.75)
 		(end 193.775 70.55)
@@
 	)
 	(segment
-		(start 184.625 70.75)
-		(end 185.075 71.2)
-		(width 0.2)
-		(layer "F.Cu")
-		(net "BAT+")
-	)
-	(segment
 		(start 184.125 70.25)
 		(end 185.075 71.2)
@@
 	)
 	(segment
+		(start 184.625 69.575)
+		(end 184.125 69.575)
+		(width 0.2)
+		(layer "F.Cu")
+		(net "BAT+")
+	)
+	(segment
 		(start 190.575 68.75)
 		(end 188.125 71.2)
@@
 	)
 	(segment
+		(start 184.63 70.755)
+		(end 185.075 71.2)
+		(width 0.2)
+		(layer "F.Cu")
+		(net "BAT+")
+	)
+	(segment
 		(start 232.962352 69.75)
 		(end 233.262352 69.45)
@@
 	)
 	(segment
-		(start 225.660994 56.953153)
-		(end 225.660994 56.760994)
+		(start 225.5 56.42)
+		(end 225.5 55.8)
 		(width 0.2)
 		(layer "F.Cu")
@@
 	)
 	(segment
-		(start 225.660994 56.760994)
-		(end 225.5 56.6)
+		(start 225.660994 56.580994)
+		(end 225.5 56.42)
 		(width 0.2)
 		(layer "F.Cu")
@@
 	)
 	(segment
-		(start 225.5 56.6)
-		(end 225.5 55.8)
+		(start 225.660994 56.953153)
+		(end 225.660994 56.580994)
 		(width 0.2)
 		(layer "F.Cu")
@@
 	)
 	(segment
+		(start 184.125 66.065)
+		(end 184.2525 65.9375)
+		(width 0.2)
+		(layer "F.Cu")
+		(net "SYS_OUT")
+	)
+	(segment
 		(start 185.8375 68.8625)
 		(end 188.5125 68.8625)
@@
 	)
 	(segment
-		(start 185.709143 65.9375)
-		(end 188.525 68.753357)
+		(start 186.1875 65.9375)
+		(end 184.2525 65.9375)
 		(width 0.2)
 		(layer "F.Cu")
@@
 	)
 	(segment
-		(start 184.8375 65.9375)
-		(end 184.910614 65.9375)
+		(start 187.375 67.125)
+		(end 187.375 67.925)
 		(width 0.2)
 		(layer "F.Cu")
@@
 	)
 	(segment
-		(start 184.910614 65.9375)
-		(end 185.709143 65.9375)
+		(start 187.375 67.925)
+		(end 188.3 68.85)
 		(width 0.2)
 		(layer "F.Cu")
@@
 	)
 	(segment
-		(start 184.625 66.65)
-		(end 184.625 66.223114)
+		(start 188.3 68.85)
+		(end 188.525 68.85)
 		(width 0.2)
 		(layer "F.Cu")
@@
 	)
 	(segment
-		(start 184.625 66.223114)
-		(end 184.910614 65.9375)
+		(start 184.625 66.65)
+		(end 184.625 65.9375)
 		(width 0.2)
 		(layer "F.Cu")
@@
 	(segment
 		(start 184.125 66.65)
-		(end 184.8375 65.9375)
+		(end 184.125 66.065)
 		(width 0.2)
 		(layer "F.Cu")
@@
 	)
 	(segment
-		(start 188.525 68.753357)
-		(end 188.525 68.85)
+		(start 186.1875 65.9375)
+		(end 187.375 67.125)
 		(width 0.2)
 		(layer "F.Cu")
